File: hardware/controller/controller.kicad_pcb (KiCad board)
At the start: 4 copper layers, 59 x 51 mm, 74 parts, among them J1 Conn_01x02_Pin, J11 Barrel_Jack, J12 USB_C_Receptacle_USB2.0_14P, J2 Conn_01x02_Pin, J3 Conn_01x02_Pin, J5 Screw_Terminal_01x02, J6 Screw_Terminal_01x02, J7 Conn_01x04_Pin, J8 Conn_01x04_Pin, U1 ESP32-C3-MINI-1, U2 MAX31855KASA, U3 MAX31855KASA, U4 MAX31855KASA, U5 TPS2121RUXR, U6 TPS1H200AQDGNRQ1, U7 LP2985-3.3, U8 AP63203WU

Commit message: Move output terminals, resize board
Parts:
- removed TP6: TestPoint, TestPoint:TestPoint_THTPad_2.0x2.0mm_Drill1.0mm
- moved U6 10.0 mm to (159.0, 104.6), turned to 180 degrees
- moved R3 8.33 mm to (154.8, 91.2), turned to 180 degrees
- moved D2 7.26 mm to (158.3, 91.2), turned to 0 degrees
- moved J6 6.51 mm to (157.7, 112.6)
- moved C1 3.98 mm to (154.7, 104.7), turned to -90 degrees
- moved J5 3.97 mm to (157.6, 100.2)
- moved TP4 3.82 mm to (160.0, 79.8)
- moved TP5 3.34 mm to (160.0, 82.8)
- moved TP1 2.29 mm to (121.7, 116.8)
- moved TP2 2.29 mm to (117.9, 116.8)
- moved TP3 2.29 mm to (114.0, 116.8)
- moved H1 2.00 mm to (161.8, 74.5)
- moved H4 2.00 mm to (161.8, 120.5)
Connections:
- U6 pad 3: Net-(U6-~{FAULT}) -> unconnected-(U6-~{FAULT}-Pad3)
Routing:
- net /Microcontroller/HEATER: track 61.8 -> 66.4 mm
- net Net-(U6-~{FAULT}): track 4.32 -> 0.00 mm
- net Net-(J6-Pin_2): track 9.46 -> 5.18 mm
- net Net-(D3-A): track 38.9 -> 34.8 mm
- net +12V: track 94.7 -> 97.7 mm
- net GND: track 94.8 -> 97.7 mm, vias 51 -> 49
- net VBUS: track 37.8 -> 40.1 mm
- net Net-(D4-A): track 38.8 -> 36.9 mm
- net Net-(D2-K): track 3.08 -> 1.68 mm
Other:
- board size 59 x 51 mm -> 57 x 51 mm
