File: hardware/controller/mcu.kicad_sch (KiCad schematic)
At the start: 25 parts, among them J12 USB_C_Receptacle_USB2.0_14P, J5 Screw_Terminal_01x02, J6 Screw_Terminal_01x02, U1 ESP32-C3-MINI-1, U6 TPS1H200AQDGNRQ1

Commit message: Move output terminals, resize board
Parts:
- removed TP6: TestPoint, TestPoint:TestPoint_THTPad_2.0x2.0mm_Drill1.0mm, symbol Connector:TestPoint
Connections:
- no-connect marks 5 -> 6
Changed lines of the file:
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@@
 	)
 	(no_connect
+		(at 62.23 132.08)
+	)
+	(no_connect
 		(at 173.99 113.03)
 	)
@@
 	(wire
 		(pts
-			(xy 54.61 132.08) (xy 62.23 132.08)
-		)
-		(stroke
-			(width 0)
-			(type default)
-		)
-	)
-	(wire
-		(pts
 			(xy 175.26 74.93) (xy 189.23 74.93)
 		)
@@
 					(unit 1)
 				)
-			)
-		)
-	)
-	(symbol
-		(lib_id "Connector:TestPoint")
-		(at 54.61 132.08 0)
-		(unit 1)
-		(exclude_from_sim no)
-		(in_bom no)
-		(on_board yes)
-		(dnp no)
-		(property "Reference" "TP6"
-			(at 53.594 127 90)
-			(effects
-				(font
-					(size 1.27 1.27)
-				)
-				(justify left)
-			)
-		)
-		(property "Value" "TestPoint"
-			(at 56.134 127 90)
-			(effects
-				(font
-					(size 1.27 1.27)
-				)
-				(justify left)
-			)
-		)
-		(property "Footprint" "TestPoint:TestPoint_THTPad_2.0x2.0mm_Drill1.0mm"
-			(at 59.69 132.08 0)
-			(effects
-				(font
-					(size 1.27 1.27)
-				)
-				(hide yes)
-			)
-		)
-		(property "Datasheet" "~"
-			(at 59.69 132.08 0)
-			(effects
-				(font
-					(size 1.27 1.27)
-				)
-				(hide yes)
-			)
-		)
-		(property "Description" "test point"
-			(at 54.61 132.08 0)
-			(effects
-				(font
-					(size 1.27 1.27)
-				)
-				(hide yes)
-			)
-		)
-		(pin "1"
-		)
-		(instances
-			(project "controller"
-				(path "/3ee12552-bbaf-4643-8241-99077a41063f/0cb4d016-03f6-42de-b902-af7c075bf798"
-					(reference "TP6")
-					(unit 1)
-				)
